File: KiCAD/analog-front-end/_autosave-emg-analog-front-end.kicad_sch (KiCad schematic)
At the start: 42 parts, among them J1 Conn_01x03, J2 Conn_01x04_Female, J3 Conn_01x04_Female, U1 AD620, U6 AD8619ARUZ-REEL

Commit message: modifying the pcb for new electrode placement and replacing op amps
Parts:
- U1: renamed from U?; footprint (none) -> Package_SO:SOIC-8_3.9x4.9mm_P1.27mm
- gave numbers to parts that had none: 5
- renumbered C12 to C1, C8 to C10, C9 to C13, C10 to C14, C11 to C15, C13 to C2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
Connections:
- net -VDD: now also C11.1
