File: KiCAD/analog-front-end/_autosave-emg-analog-front-end.kicad_sch (KiCad schematic)
At the start: 48 parts, among them J1 Conn_01x03, J2 Conn_01x05_Female, J3 Conn_01x05_Female, U1 LMC6482, U2 AD620, U3 AD8619ARUZ-REEL, U4 MAX1697REUT+T

Commit message: DRC passing, should be all good for starting fab files
Parts:
- gave numbers to parts that had none: 3
Changed lines of the file:
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@@
   (symbol (lib_id "Device:R_US") (at 41.1226 49.0728 0) (unit 1)
     (in_bom yes) (on_board yes)
-    (property "Reference" "R?" (id 0) (at 45.0088 50.1904 0)
+    (property "Reference" "R17" (id 0) (at 45.0088 50.1904 0)
       (effects (font (size 1.27 1.27)) (justify right))
     )
@@
   (symbol (lib_id "Device:R_US") (at 29.7688 43.0022 0) (unit 1)
     (in_bom yes) (on_board yes)
-    (property "Reference" "R?" (id 0) (at 33.655 44.1198 0)
+    (property "Reference" "R16" (id 0) (at 33.655 44.1198 0)
       (effects (font (size 1.27 1.27)) (justify right))
     )
@@
   (symbol (lib_id "Device:R_US") (at 23.5458 58.8772 180) (unit 1)
     (in_bom yes) (on_board yes)
-    (property "Reference" "R?" (id 0) (at 19.6596 57.7596 0)
+    (property "Reference" "R15" (id 0) (at 19.6596 57.7596 0)
       (effects (font (size 1.27 1.27)) (justify right))
     )
@@
       (reference "R14") (unit 1) (value "100k") (footprint "Resistor_SMD:R_0402_1005Metric")
     )
+    (path "/cd10a77e-9039-48e1-88f1-30e6cff9af6c"
+      (reference "R15") (unit 1) (value "0") (footprint "Resistor_SMD:R_0402_1005Metric")
+    )
+    (path "/65150bdc-d09b-4448-a56e-d5e76ca3603c"
+      (reference "R16") (unit 1) (value "0") (footprint "Resistor_SMD:R_0402_1005Metric")
+    )
     (path "/1f7daf2e-b380-4470-8713-5d02034b5ee9"
-      (reference "R?") (unit 1) (value "0") (footprint "Resistor_SMD:R_0402_1005Metric")
-    )
-    (path "/65150bdc-d09b-4448-a56e-d5e76ca3603c"
-      (reference "R?") (unit 1) (value "0") (footprint "Resistor_SMD:R_0402_1005Metric")
-    )
-    (path "/cd10a77e-9039-48e1-88f1-30e6cff9af6c"
-      (reference "R?") (unit 1) (value "0") (footprint "Resistor_SMD:R_0402_1005Metric")
+      (reference "R17") (unit 1) (value "0") (footprint "Resistor_SMD:R_0402_1005Metric")
     )
     (path "/268f0419-4fd4-4bd7-b6a2-6e801c0c7a82"
