File: KiCAD/analog-front-end/_autosave-emg-analog-front-end.kicad_sch (KiCad schematic)
At the start: 46 parts, among them J1 Conn_01x03, J2 Conn_01x04_Female, J3 Conn_01x04_Female, U1 AD620, U2 LMC6492, U3 LMC6492, U4 LMC6492

Commit message: v3 layout done
Parts:
- gave numbers to parts that had none: 3
Changed lines of the file:
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@@
   (symbol (lib_id "power:VDD") (at 119.0498 166.3192 0) (unit 1)
     (in_bom yes) (on_board yes) (fields_autoplaced)
-    (property "Reference" "#PWR?" (id 0) (at 119.0498 170.1292 0)
+    (property "Reference" "#PWR0102" (id 0) (at 119.0498 170.1292 0)
       (effects (font (size 1.27 1.27)) hide)
     )
@@
   (symbol (lib_id "pspice:C") (at 110.236 175.8696 90) (unit 1)
     (in_bom yes) (on_board yes)
-    (property "Reference" "C?" (id 0) (at 108.7628 168.4528 90)
+    (property "Reference" "C18" (id 0) (at 108.7628 168.4528 90)
       (effects (font (size 1.27 1.27)) (justify right))
     )
@@
   (symbol (lib_id "MAX1697REUT_T:MAX1697REUT+T") (at 138.7602 175.8696 0) (unit 1)
     (in_bom yes) (on_board yes) (fields_autoplaced)
-    (property "Reference" "U?" (id 0) (at 138.7602 160.02 0))
+    (property "Reference" "U5" (id 0) (at 138.7602 160.02 0))
     (property "Value" "MAX1697REUT+T" (id 1) (at 138.7602 162.56 0))
     (property "Footprint" "SOT95P280X145-6N" (id 2) (at 138.7602 175.8696 0)
@@
   (symbol (lib_id "pspice:C") (at 163.6014 175.8188 180) (unit 1)
     (in_bom yes) (on_board yes)
-    (property "Reference" "C?" (id 0) (at 155.6004 173.9138 0)
+    (property "Reference" "C19" (id 0) (at 155.6004 173.9138 0)
       (effects (font (size 1.27 1.27)) (justify right))
     )
@@
   (symbol (lib_id "power:GND") (at 163.6014 185.0898 0) (unit 1)
     (in_bom yes) (on_board yes) (fields_autoplaced)
-    (property "Reference" "#PWR?" (id 0) (at 163.6014 191.4398 0)
+    (property "Reference" "#PWR0103" (id 0) (at 163.6014 191.4398 0)
       (effects (font (size 1.27 1.27)) hide)
     )
@@
     )
     (path "/20926577-f654-40a7-9c84-328b7072dd5d"
-      (reference "#PWR?") (unit 1) (value "VDD") (footprint "")
+      (reference "#PWR0102") (unit 1) (value "VDD") (footprint "")
     )
     (path "/f060f5b3-0525-4199-87f4-b0a9675e2627"
-      (reference "#PWR?") (unit 1) (value "GND") (footprint "")
+      (reference "#PWR0103") (unit 1) (value "GND") (footprint "")
     )
     (path "/d1edc5ae-c074-46b3-9795-91dd6414ec52"
@@
     )
     (path "/414cf7d5-6e72-434b-a754-58df4dd52df8"
-      (reference "C?") (unit 1) (value "1uF") (footprint "Capacitor_SMD:C_0402_1005Metric")
+      (reference "C18") (unit 1) (value "1uF") (footprint "Capacitor_SMD:C_0402_1005Metric")
     )
     (path "/dfbef705-6c54-43aa-a161-d6449927b091"
-      (reference "C?") (unit 1) (value "1uF") (footprint "Capacitor_SMD:C_0402_1005Metric")
+      (reference "C19") (unit 1) (value "1uF") (footprint "Capacitor_SMD:C_0402_1005Metric")
     )
     (path "/c46d5690-7295-47f7-a0c8-1058116b8405"
@@
     )
     (path "/97e59e1c-e5d2-4d05-a9fb-968536188e0f"
-      (reference "U?") (unit 1) (value "MAX1697REUT+T") (footprint "SOT95P280X145-6N")
-    )
-  )
+      (reference "U5") (unit 1) (value "MAX1697REUT+T") (footprint "SOT95P280X145-6N")
+    )
+  )
