File: KiCAD/analog-front-end/_autosave-emg-analog-front-end.kicad_pcb (KiCad board)
At the start: 2 copper layers, 42 x 20 mm, 49 parts, among them J1 Conn_01x03, J2 Conn_01x05_Female, J3 Conn_01x05_Female, U1 LMC6482, U2 AD620, U3 AD8619ARUZ-REEL, U4 MAX1697REUT+T

Commit message: DRC passing, should be all good for starting fab files
Parts:
- moved R8 0.82 mm to (11.8, 16.2)
- moved U4 0.67 mm to (7.92, 15.4)
- moved C16 0.67 mm to (7.32, 18.0)
- moved R14 0.36 mm to (12.3, 14.2), turned to 0 degrees
Routing:
- net GND: track 52.9 -> 65.1 mm, vias 6 -> 7
- net VDD: track 58.8 -> 60.4 mm, vias 5 -> 4
- net Net-(R14-Pad1): track 3.29 -> 4.35 mm
- net -VDD: track 67.0 -> 66.4 mm, vias 3 -> 6
