File: KiCAD/analog-front-end/_autosave-emg-analog-front-end.kicad_pcb (KiCad board)
At the start: 4 copper layers, 42 x 18 mm, 47 parts, among them J1 Conn_01x03, J2 Conn_01x04_Female, J3 Conn_01x04_Female, U1 AD620, U2 LMC6492, U3 LMC6492, U4 LMC6492, U5 MAX1697REUT+T

Commit message: v3 layout done
Parts:
- moved G*** 24.0 mm to (32.1, 14.6)
- moved TP1 14.9 mm to (35.1, 16.6)
- moved TP2 13.6 mm to (12.2, 16.6)
Routing:
- net AOUT_CH0: track 12.6 -> 26.8 mm
- net -VDD: track 10.9 -> 21.1 mm
- net GND: track 29.2 -> 37.0 mm, vias 13 -> 14
- net VDD: track 20.2 -> 24.4 mm, vias 5 -> 7
- added copper zone on F.Cu, net -VDD
- removed copper zone on B.Cu, net -VDD
Other:
- board text added: "-VDD"
- board text added: "GND"
- board text added: "OUT"
- board text added: "VDD"
