File: KiCAD/analog-front-end/emg-analog-front-end.kicad_pcb (KiCad board)
At the start: 4 copper layers, 42 x 18 mm, 47 parts, among them J1 Conn_01x03, J2 Conn_01x04_Female, J3 Conn_01x04_Female, U1 AD620, U2 LMC6492, U3 LMC6492, U4 LMC6492, U5 MAX1697REUT+T

Commit message: adding production files
Parts:
- removed J3: Conn_01x04_Female, Connector_PinHeader_1.27mm:PinHeader_1x04_P1.27mm_Vertical
- added J4: Conn_01x08_Female, Connector_PinHeader_1.27mm:PinHeader_1x08_P1.27mm_Vertical, F.Cu at (20.1, 1.90)
- G***: moved to B.Cu
- J2: value Conn_01x04_Female -> Conn_01x08_Female; footprint Connector_PinHeader_1.27mm:PinHeader_1x04_P1.27mm_Vertical -> Connector_PinHeader_1.27mm:PinHeader_1x08_P1.27mm_Vertical
- moved G*** 46.0 mm to (8.60, 8.40), turned to 180 degrees
- moved TP1 18.7 mm to (32.1, 13.9)
- moved J2 12.9 mm to (20.1, 14.1)
- moved TP2 12.6 mm to (7.40, 14.2)
- moved C18 4.50 mm to (12.9, 14.2), turned to 180 degrees
- moved C2 3.80 mm to (22.2, 8.20), turned to 90 degrees
- moved C10 3.71 mm to (15.9, 2.90)
- moved R12 3.57 mm to (14.9, 2.90)
- moved R13 3.56 mm to (17.3, 1.37)
- moved C11 3.56 mm to (15.3, 1.37)
- moved R3 3.46 mm to (22.7, 9.70)
- moved R9 2.67 mm to (12.9, 2.91), turned to -90 degrees
- moved C17 2.52 mm to (32.6, 11.9), turned to 0 degrees
- moved U4 2.21 mm to (35.4, 8.50)
- moved R6 1.86 mm to (12.2, 12.1)
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Connections:
- J2 pad 4: -VDD -> AOUT_CH1
Routing:
- net -VDD: track 10.9 -> 43.9 mm, vias 0 -> 7
- net /HPF_OUT_CH0: track 4.79 -> 19.2 mm, vias 0 -> 2
- net AOUT_CH3: track 0.00 -> 12.6 mm, vias 0 -> 1
- net NOTCH_OUT_CH0: track 20.5 -> 32.9 mm, vias 3 -> 2
- net AOUT_CH1: track 0.00 -> 12.2 mm, vias 0 -> 1
- net AOUT_CH4: track 0.00 -> 12.2 mm, vias 0 -> 1
- net AOUT_CH2: track 0.00 -> 12.2 mm, vias 0 -> 1
- net AOUT_CH0: track 12.6 -> 23.8 mm, vias 2 -> 1
- net GND: track 29.2 -> 37.0 mm, vias 13 -> 11
- net VDD: track 20.2 -> 27.8 mm, vias 5 -> 6
- net /LPF_IN-_CH0: track 9.51 -> 5.62 mm
- net SK00: track 21.7 -> 18.9 mm
- net Net-(C11-Pad1): track 4.17 -> 2.08 mm
- net SK01: track 2.20 -> 4.22 mm
- net Net-(C18-Pad2): track 8.07 -> 9.97 mm, vias 0 -> 2
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- added copper zone on F.Cu, net -VDD
- removed copper zone on B.Cu, net -VDD
Other:
- board size 42 x 18 mm -> 39.6 x 16.3 mm
- board text removed: "HPF"
- board text removed: "LPF"
