File: KiCAD/analog-front-end/emg-analog-front-end.kicad_sch (KiCad schematic)
At the start: 46 parts, among them J1 Conn_01x03, J2 Conn_01x04_Female, J3 Conn_01x04_Female, U1 AD620, U2 LMC6492, U3 LMC6492, U4 LMC6492

Commit message: adding production files
Parts:
- removed J2, J3: Conn_01x04_Female, Connector_PinHeader_1.27mm:PinHeader_1x04_P1.27mm_Vertical, symbol Connector:Conn_01x04_Female
- added J2, J4: Conn_01x08_Female, Connector_PinHeader_1.27mm:PinHeader_1x08_P1.27mm_Vertical, symbol Connector:Conn_01x08_Female
- gave numbers to parts that had none: 3
Connections:
- net -VDD: now also J2.8 (Pin_8), J4.8 (Pin_8)
- net AOUT_CH0: now also J2.3 (Pin_3), J4.3 (Pin_3)
- net GND: now also J2.1 (Pin_1), J4.1 (Pin_1)
- net VDD: now also J2.2 (Pin_2), J4.2 (Pin_2)
- new net AOUT_CH1: J2.4 (Pin_4), J4.4 (Pin_4)
- new net AOUT_CH2: J2.5 (Pin_5), J4.5 (Pin_5)
- new net AOUT_CH3: J2.6 (Pin_6), J4.6 (Pin_6)
- new net AOUT_CH4: J2.7 (Pin_7), J4.7 (Pin_7)
Other:
- moved on the sheet: R10, R11, R7, R8, U3A, U3B
